File: Eletrica/placacomLed/placacomLed.kicad_sch (KiCad schematic)
At the start: 3 parts, among them J1 Screw_Terminal_01x02

Commit message: Estrutura2
Parts:
- D1: footprint (none) -> LED_THT:LED_D3.0mm
- J1: footprint (none) -> TerminalBlock_4Ucon:TerminalBlock_4Ucon_1x02_P3.50mm_Horizontal
- R1: footprint (none) -> Resistor_THT:R_Axial_DIN0411_L9.9mm_D3.6mm_P12.70mm_Horizontal
Changed lines of the file:
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@@
       (effects (font (size 1.27 1.27)) hide)
     )
-    (property "Footprint" "" (at 132.08 102.87 0)
+    (property "Footprint" "LED_THT:LED_D3.0mm" (at 132.08 102.87 0)
       (effects (font (size 1.27 1.27)) hide)
     )
@@
       (effects (font (size 1.27 1.27)) hide)
     )
-    (property "Footprint" "" (at 140.97 104.648 90)
+    (property "Footprint" "Resistor_THT:R_Axial_DIN0411_L9.9mm_D3.6mm_P12.70mm_Horizontal" (at 140.97 104.648 90)
       (effects (font (size 1.27 1.27)) hide)
     )
@@
       (effects (font (size 1.27 1.27)) (justify left) hide)
     )
-    (property "Footprint" "" (at 151.13 100.33 0)
+    (property "Footprint" "TerminalBlock_4Ucon:TerminalBlock_4Ucon_1x02_P3.50mm_Horizontal" (at 151.13 100.33 0)
       (effects (font (size 1.27 1.27)) hide)
     )
